File: hardware/aether-carrier.kicad_sch (KiCad schematic)
At the start: 0 parts

Commit message: engineering: Rev B zero-interference CAD, sealed STL meshes and carrier corrections
Other:
- title: Aether Orb - Rev A carrier -> Aether Orb - Rev B carrier
